Commit message: change colors of bots

File: urdf/turtlebot3_burger.urdf.xacro (robot description, xacro)
@@ -3,4 +3,5 @@
   <xacro:include filename="$(find turtlebot3_description)/urdf/common_properties.xacro"/>
   <xacro:include filename="$(find turtlebot3_description)/urdf/turtlebot3_burger.gazebo.xacro"/>
+  <xacro:arg name="chassis_color" default="DarkGrey"/>
   <link name="base_footprint"/>
   <joint name="base_joint" type="fixed">
@@ -15,5 +16,5 @@
         <mesh filename="package://turtlebot3_description/meshes/bases/burger_base.stl" scale="0.001 0.001 0.001"/>
       </geometry>
-      <material name="light_black"/>
+      <material name="$(arg chassis_color)"/>
     </visual>
     <collision>
@@ -31,4 +32,7 @@
     </inertial>
   </link>
+  <gazebo reference="base_link">
+    <material>Gazebo/$(arg chassis_color)</material>
+  </gazebo>
   <joint name="wheel_left_joint" type="continuous">
     <parent link="base_link"/>

File: urdf/turtlebot3_waffle.urdf.xacro (robot description, xacro)
@@ -8,4 +8,5 @@
   <xacro:property name="r200_cam_depth_offset" value="0.01"/>
   <link name="base_footprint"/>
+  <xacro:arg name="chassis_color" default="DarkGrey"/>
   <joint name="base_joint" type="fixed">
     <parent link="base_footprint"/>
@@ -35,4 +36,7 @@
     </inertial>
   </link>
+  <gazebo reference="base_link">
+    <material>Gazebo/$(arg chassis_color)</material>
+  </gazebo>
   <joint name="wheel_left_joint" type="continuous">
     <parent link="base_link"/>
